Commit message: nano_atom_description: Support for ov5647 camera added

File: nano_atom_common/nano_atom_description/urdf/accessories/ov5647_support.urdf.xacro (robot description, xacro)
@@ -1,10 +1,10 @@
 <?xml version="1.0"?>
-<robot name="structure_kinect_support" xmlns:xacro="http://www.ros.org/wiki/xacro">
-  <xacro:macro name ="structure_kinect_support" params="prefix parent *origin">
-    <link name="${prefix}_link">
+<robot name="ov5647_support" xmlns:xacro="http://www.ros.org/wiki/xacro">
+  <xacro:macro name ="ov5647_support" params="prefix parent *origin">
+    <link name="${prefix}link">
         <collision>
         <origin xyz="0 0 0" rpy="0 0 0"/>
         <geometry>
-            <mesh filename="package://nano_atom_description/meshes/accessories/kinect_support_simple.stl" />
+            <mesh filename="package://nano_atom_description/meshes/accessories/ov5647_support.stl" />
         </geometry>
         </collision>
@@ -12,5 +12,5 @@
         <origin xyz="0 0 0" rpy="0 0 0"/>
         <geometry>
-            <mesh filename="package://nano_atom_description/meshes/accessories/kinect_support.dae" />
+            <mesh filename="package://nano_atom_description/meshes/accessories/ov5647_support.stl" />
         </geometry>
         </visual>
@@ -24,5 +24,5 @@
         <xacro:insert_block name="origin" />
         <parent link="${parent}"/>
-        <child link="${prefix}_link"/>
+        <child link="${prefix}link"/>
     </joint>
   </xacro:macro>
