Commit message: nano_atom_description: xacro robot updated

File: nano_atom_common/nano_atom_description/robots/nano_atom_std.urdf.xacro (robot description, xacro)
@@ -9,4 +9,5 @@
   <xacro:arg name="use_central_cube"  default="false"            />
   <xacro:arg name="use_sim"           default="true"             />
+  <xacro:arg name="gpu_laser_sim"     default="true"             />
   <xacro:arg name="footprint_frame"   default="$(arg prefix)base_footprint" />
   <xacro:arg name="base_frame"        default="$(arg prefix)base_link"      />
@@ -18,10 +19,10 @@
   <xacro:include filename="$(find nano_atom_description)/urdf/wheels/rubber_wheel.urdf.xacro" />
   <xacro:include filename="$(find nano_atom_description)/urdf/wheels/caster_wheel.urdf.xacro" />
-  <!-- Import nano_atom accessories: kinect support accesory -->
-  <xacro:include filename="$(find nano_atom_description)/urdf/accesories/kinect_support.urdf.xacro" />
+  <!-- Import nano_atom accessories: kinect support accessory -->
+  <xacro:include filename="$(find nano_atom_description)/urdf/accessories/ov5647_support.urdf.xacro" />
   <!-- Import nano_atom sensors: ydlidar x2 -->
   <xacro:include filename="$(find roboticarts_sensors)/urdf/ydlidar_x2.urdf.xacro" />
-  <!-- Import nano_atom sensors: kinect camera -->
-  <xacro:include filename="$(find roboticarts_sensors)/urdf/kinect.urdf.xacro" />
+  <!-- Import nano_atom sensors: ov5647 camera -->
+  <xacro:include filename="$(find roboticarts_sensors)/urdf/ov5647.urdf.xacro" />
   <!-- Import nano_atom sensors: imu sensor -->
   <xacro:include filename="$(find roboticarts_sensors)/urdf/imu.urdf.xacro" />
@@ -53,10 +54,10 @@
 	<xacro:property name="wheel_offset_y" value="0.04519" />
 	<xacro:property name="wheel_offset_z" value="0.005" />
-  <xacro:omni_wheel prefix="$(arg prefix)right_" parent ="$(arg base_frame)" type="right">
+  <xacro:rubber_wheel prefix="$(arg prefix)right_" parent ="$(arg base_frame)" type="right">
   	<origin xyz="${wheel_offset_x} -${wheel_offset_y} +${wheel_offset_z}" rpy="0 0 0"/>
-  </xacro:omni_wheel>
-  <xacro:omni_wheel prefix="$(arg prefix)left_" parent ="$(arg base_frame)" type="left">
+  </xacro:rubber_wheel>
+  <xacro:rubber_wheel prefix="$(arg prefix)left_" parent ="$(arg base_frame)" type="left">
   	<origin xyz="${wheel_offset_x} +${wheel_offset_y} +${wheel_offset_z}" rpy="0 0 0"/>
-  </xacro:omni_wheel>
+  </xacro:rubber_wheel>
   <!-- Caster parameters -->
 	<xacro:property name="caster_offset_x" value="0.04746" />
@@ -69,8 +70,9 @@
   	<origin xyz="-${caster_offset_x} +${caster_offset_y} -${caster_offset_z}" rpy="0 0 0"/>
   </xacro:caster_wheel>
-<!-- - - - - - - - - - - - - - ACCESORIES DEFINITION  - - - - - - - - - - - - - -->
+<!-- - - - - - - - - - - - - - ACCESSORIES DEFINITION  - - - - - - - - - - - - - -->
   <!-- ydlidar x2 lidar sensor -->
   <xacro:if value="$(arg use_front_laser)">
-    <xacro:sensor_ydlidar_x2 prefix="$(arg prefix)front_laser_" parent="$(arg base_frame)" prefix_topic="front_laser/scan" use_sim="$(arg use_sim)" >
+    <xacro:sensor_ydlidar_x2 prefix="$(arg prefix)front_laser_" parent="$(arg base_frame)" prefix_topic="front_laser/scan" use_sim="$(arg use_sim)"
+                             gpu_sim="$(arg gpu_laser_sim)" >
       <origin xyz="0 0 0.08538" rpy="0 0 0"/>
     </xacro:sensor_ydlidar_x2>
@@ -82,10 +84,14 @@
     </xacro:sensor_imu>
   </xacro:if>
-  <!-- kinect camera
+  <!-- Front Camera -->
   <xacro:if value="$(arg use_front_camera)">
-    <xacro:sensor_kinect prefix="$(arg prefix)front_camera_" parent ="$(arg base_frame)" prefix_topic="front_camera" use_sim="$(arg use_sim)" >
-      <origin xyz="-0.05 0 0.27" rpy="0 0 0"/>
-    </xacro:sensor_kinect>
+    <!-- ov5647 support -->
+    <xacro:ov5647_support prefix="$(arg prefix)support_camera_" parent ="$(arg base_frame)">
+      <origin xyz="0.064 0 0.0715" rpy="0 0 0"/>
+    </xacro:ov5647_support>
+    <!-- ov5647 camera -->
+    <xacro:sensor_ov5647 prefix="$(arg prefix)front_camera_" parent ="$(arg prefix)support_camera_link" prefix_topic="front_camera" use_sim="$(arg use_sim)" >
+      <origin xyz="0.002 0 -0.017" rpy="0 0 0"/>
+    </xacro:sensor_ov5647>
   </xacro:if>
-  -->
 </robot>

File: nano_atom_common/nano_atom_description/urdf/wheels/rubber_wheel.urdf.xacro (robot description, xacro)
@@ -34,5 +34,5 @@
   </xacro:macro>
 <!-- - - - - - - - - - - - - - WHEEL DEFINITION - - - - - - - - - - - - - -->
-  <xacro:macro name ="omni_wheel" params = "prefix parent *origin type">
+  <xacro:macro name ="rubber_wheel" params = "prefix parent *origin type">
     <!-- wheel & base joint-->
     <joint name="${prefix}wheel_joint" type="continuous">
@@ -45,16 +45,16 @@
     <link name="${prefix}wheel_link">
       <inertial>
-        <origin_selector wheel = "${type}" />
+        <xacro:origin_selector wheel = "${type}" />
         <mass value="${wheel_mass}" />
-        <inertia_selector wheel = "${type}" />
+        <xacro:inertia_selector wheel = "${type}" />
       </inertial>
       <visual>
         <origin xyz="0 0 0" rpy="0 0 0" />
         <geometry>
-          <mesh_selector wheel = "${type}"  extension = ".stl" />
+          <xacro:mesh_selector wheel = "${type}"  extension = ".stl" />
         </geometry>
       </visual>
       <collision>
-        <origin_selector wheel = "${type}" />
+        <xacro:origin_selector wheel = "${type}" />
         <geometry>
           <cylinder length="${wheel_width}" radius="${wheel_radius}" />
