Commit message: base/nano_atom_description: Add basic sensors and colors

File: src/base/nano_atom_description/robots/nano_atom_std.urdf.xacro (robot description, xacro)
@@ -3,5 +3,5 @@
 <!-- - - - - - - - - - - - - - GLOBAL ARGUMENTS - - - - - - - - - - - - - -->
   <xacro:arg name="robot_id"            default="robot" />
-  <xacro:arg name="prefix"              default="$(arg robot_id)_" />
+  <xacro:arg name="prefix"              default="$(arg robot_id)/" />
   <xacro:arg name="controller_sim_path" default="$(find ${nano_atom_control})/config/diff_controller.yaml" />
   <xacro:arg name="hardware_path"       default="$(find ${nano_atom_hardware})/config/hardware.yaml" />
@@ -23,13 +23,11 @@
   <!-- Import nano_atom accessories: kinect support accessory -->
   <xacro:include filename="$(find nano_atom_description)/urdf/accessories/ov5647_support.urdf.xacro" />
-  <!-- Import nano_atom sensors: ydlidar x2
-  <xacro:include filename="$(find roboticarts_sensors)/urdf/ydlidar_x2.urdf.xacro" />
+  <!-- Import nano_atom sensors: ydlidar x2 -->
+  <xacro:include filename="$(find nano_atom_description)/urdf/devices/ydlidar_x2.urdf.xacro" />
+  <!-- Import nano_atom sensors: ov5647 camera
+  <xacro:include filename="$(find nano_atom_description)/urdf/devices/ov5647.urdf.xacro" />
   -->
-  <!-- Import nano_atom sensors: ov5647 camera
-  <xacro:include filename="$(find roboticarts_sensors)/urdf/ov5647.urdf.xacro" />
-  -->
-  <!-- Import nano_atom sensors: imu sensor
-  <xacro:include filename="$(find roboticarts_sensors)/urdf/imu.urdf.xacro" />
-  -->
+  <!-- Import nano_atom sensors: imu sensor -->
+  <xacro:include filename="$(find nano_atom_description)/urdf/devices/imu.urdf.xacro" />
   <!-- Import nano_atom control -->
   <xacro:include filename="$(find nano_atom_description)/urdf/controllers/diff.ros2_control.urdf.xacro" />
@@ -76,5 +74,5 @@
   </xacro:caster_wheel>
 <!-- - - - - - - - - - - - - - ACCESSORIES DEFINITION  - - - - - - - - - - - - - -->
-  <!-- ydlidar x2 lidar sensor
+  <!-- ydlidar x2 lidar sensor -->
   <xacro:if value="$(arg use_front_laser)">
     <xacro:sensor_ydlidar_x2 prefix="$(arg prefix)front_laser_" parent="$(arg base_frame)" prefix_topic="front_laser/scan" use_sim="$(arg use_sim)"
@@ -83,6 +81,5 @@
     </xacro:sensor_ydlidar_x2>
   </xacro:if>
--->
-  <!-- IMU Sensor
+  <!-- IMU Sensor -->
   <xacro:if value="$(arg use_imu)">
     <xacro:sensor_imu prefix="$(arg prefix)imu_" parent ="$(arg base_frame)" prefix_topic="imu/data" use_sim="$(arg use_sim)" >
@@ -90,5 +87,4 @@
     </xacro:sensor_imu>
   </xacro:if>
-  -->
   <!-- Front Camera
   <xacro:if value="$(arg use_front_camera)">

File: src/base/nano_atom_description/urdf/bases/nano_atom_base.urdf.xacro (robot description, xacro)
@@ -25,4 +25,7 @@
           <mesh filename="package://nano_atom_description/meshes/bases/nano_atom_chassis.stl" />
         </geometry>
+        <material name="red">
+          <color rgba="1.0 0.0 0.0 1.0"/>
+        </material>
       </visual>
       <collision>

File: src/base/nano_atom_description/urdf/wheels/rubber_wheel.urdf.xacro (robot description, xacro)
@@ -54,4 +54,7 @@
           <xacro:mesh_selector wheel = "${type}"  extension = ".stl" />
         </geometry>
+        <material name="dark_gray">
+          <color rgba="0.2 0.2 0.2 1.0"/>
+        </material>
       </visual>
       <collision>

Commit message: base/nano_atom_description: Update and improve meshes

File: src/base/nano_atom_description/robots/nano_atom_std.urdf.xacro (robot description, xacro)
@@ -66,5 +66,5 @@
 	<xacro:property name="caster_offset_x" value="0.04746" />
 	<xacro:property name="caster_offset_y" value="0.0" />
-	<xacro:property name="caster_offset_z" value="0.01075" />
+	<xacro:property name="caster_offset_z" value="0.0025" />
   <xacro:caster_wheel prefix="$(arg prefix)front_" parent ="$(arg base_frame)">
   	<origin xyz="+${caster_offset_x} +${caster_offset_y} -${caster_offset_z}" rpy="0 0 0"/>
@@ -78,5 +78,5 @@
     <xacro:sensor_ydlidar_x2 prefix="$(arg prefix)front_laser_" parent="$(arg base_frame)" prefix_topic="front_laser/scan" use_sim="$(arg use_sim)"
                              gpu_sim="$(arg gpu_laser_sim)" >
-      <origin xyz="0 0 0.08538" rpy="0 0 0"/>
+      <origin xyz="0 0 0.09038" rpy="0 0 0"/>
     </xacro:sensor_ydlidar_x2>
   </xacro:if>

File: src/base/nano_atom_description/urdf/bases/nano_atom_base.urdf.xacro (robot description, xacro)
@@ -23,15 +23,12 @@
         <origin xyz="0 0 0" rpy="0 0 0" />
         <geometry>
-          <mesh filename="package://nano_atom_description/meshes/bases/nano_atom_chassis.stl" />
+          <mesh filename="package://nano_atom_description/meshes/bases/nano_atom_chassis.dae" />
         </geometry>
-        <material name="red">
-          <color rgba="1.0 0.0 0.0 1.0"/>
-        </material>
       </visual>
       <collision>
-        <origin xyz="0 0 0" rpy="0 0 0" />
-        <geometry>
-           <mesh filename="package://nano_atom_description/meshes/bases/nano_atom_chassis.stl" />
-        </geometry>
+        <origin xyz="0 0 0.0415" rpy="0 0 0" />
+          <geometry>
+            <cylinder radius="0.0575" length="0.083" />
+          </geometry>
       </collision>
     </link>

File: src/base/nano_atom_description/urdf/devices/ydlidar_x2.urdf.xacro (robot description, xacro)
@@ -13,9 +13,6 @@
         <origin xyz="0 0 0" rpy="0 0 0"/>
         <geometry>
-          <mesh filename="package://nano_atom_description/meshes/devices/ydlidar_x2.stl"/>
+          <mesh filename="package://nano_atom_description/meshes/devices/ydlidar_x2.dae"/>
         </geometry>
-        <material name="dark_blue">
-          <color rgba="0.0 0.0 0.45 1.0"/>
-        </material>
       </visual>
       <inertial>

File: src/base/nano_atom_description/urdf/wheels/caster_wheel.urdf.xacro (robot description, xacro)
@@ -24,9 +24,9 @@
         <origin xyz="0 0 0" rpy="0 0 0" />
         <geometry>
-          <mesh filename="package://nano_atom_description/meshes/wheels/nano_atom_caster_wheel.stl" />
+          <mesh filename="package://nano_atom_description/meshes/wheels/nano_atom_caster_wheel.dae" />
         </geometry>
       </visual>
       <collision>
-        <origin xyz="0 0 0" rpy="0 0 0" />
+        <origin xyz="0 0 -0.00825" rpy="0 0 0" />
         <geometry>
           <sphere radius="${caster_radius}"/>

File: src/base/nano_atom_description/urdf/wheels/rubber_wheel.urdf.xacro (robot description, xacro)
@@ -52,9 +52,6 @@
         <origin xyz="0 0 0" rpy="0 0 0" />
         <geometry>
-          <xacro:mesh_selector wheel = "${type}"  extension = ".stl" />
+          <xacro:mesh_selector wheel = "${type}"  extension = ".dae" />
         </geometry>
-        <material name="dark_gray">
-          <color rgba="0.2 0.2 0.2 1.0"/>
-        </material>
       </visual>
       <collision>

Commit message: base/description: Add ov5647 camera

File: src/base/nano_atom_description/robots/nano_atom_std.urdf.xacro (robot description, xacro)
@@ -11,5 +11,4 @@
   <xacro:arg name="use_central_cube"    default="false" />
   <xacro:arg name="use_sim"             default="true" />
-  <xacro:arg name="gpu_laser_sim"       default="true" />
   <xacro:arg name="footprint_frame"     default="$(arg prefix)base_footprint" />
   <xacro:arg name="base_frame"          default="$(arg prefix)base_link" />
@@ -25,7 +24,6 @@
   <!-- Import nano_atom sensors: ydlidar x2 -->
   <xacro:include filename="$(find nano_atom_description)/urdf/devices/ydlidar_x2.urdf.xacro" />
-  <!-- Import nano_atom sensors: ov5647 camera
+  <!-- Import nano_atom sensors: ov5647 camera -->
   <xacro:include filename="$(find nano_atom_description)/urdf/devices/ov5647.urdf.xacro" />
-  -->
   <!-- Import nano_atom sensors: imu sensor -->
   <xacro:include filename="$(find nano_atom_description)/urdf/devices/imu.urdf.xacro" />
@@ -76,6 +74,5 @@
   <!-- ydlidar x2 lidar sensor -->
   <xacro:if value="$(arg use_front_laser)">
-    <xacro:sensor_ydlidar_x2 prefix="$(arg prefix)front_laser_" parent="$(arg base_frame)" prefix_topic="front_laser/scan" use_sim="$(arg use_sim)"
-                             gpu_sim="$(arg gpu_laser_sim)" >
+    <xacro:sensor_ydlidar_x2 prefix="$(arg prefix)front_laser_" parent="$(arg base_frame)" prefix_topic="front_laser/scan" use_sim="$(arg use_sim)">
       <origin xyz="0 0 0.09038" rpy="0 0 0"/>
     </xacro:sensor_ydlidar_x2>
@@ -84,18 +81,17 @@
   <xacro:if value="$(arg use_imu)">
     <xacro:sensor_imu prefix="$(arg prefix)imu_" parent ="$(arg base_frame)" prefix_topic="imu/data" use_sim="$(arg use_sim)" >
-      <origin xyz="-0.0305 0 0.036" rpy="0 0 0"/>
+      <origin xyz="-0.0305 0 0.0" rpy="0 0 0"/>
     </xacro:sensor_imu>
   </xacro:if>
-  <!-- Front Camera
+  <!-- Front Camera -->
   <xacro:if value="$(arg use_front_camera)">
-     ov5647 support
+    <!-- ov5647 support -->
     <xacro:ov5647_support prefix="$(arg prefix)support_camera_" parent ="$(arg base_frame)">
-      <origin xyz="0.064 0 0.0715" rpy="0 0 0"/>
+      <origin xyz="0.064 0 0.0815" rpy="0 0 0"/>
     </xacro:ov5647_support>
-     ov5647 camera
+    <!-- ov5647 camera -->
     <xacro:sensor_ov5647 prefix="$(arg prefix)front_camera_" parent ="$(arg prefix)support_camera_link" prefix_topic="front_camera" use_sim="$(arg use_sim)" >
       <origin xyz="0.002 0 -0.017" rpy="0 0 0"/>
     </xacro:sensor_ov5647>
   </xacro:if>
-  -->
 </robot>

File: src/base/nano_atom_description/urdf/accessories/ov5647_support.urdf.xacro (robot description, xacro)
@@ -12,5 +12,5 @@
         <origin xyz="0 0 0" rpy="0 0 0"/>
         <geometry>
-            <mesh filename="package://nano_atom_description/meshes/accessories/ov5647_support.stl" />
+            <mesh filename="package://nano_atom_description/meshes/accessories/ov5647_support.dae" />
         </geometry>
         </visual>

File: src/base/nano_atom_description/urdf/devices/ov5647.urdf.xacro (robot description, xacro)
@@ -9,5 +9,5 @@
         <origin xyz="0 0 0" rpy="0 0 0"/>
         <geometry>
-          <mesh filename="package://nano_atom_description/meshes/devices/ov5647.stl" />
+          <mesh filename="package://nano_atom_description/meshes/devices/ov5647.dae" />
         </geometry>
       </visual>
@@ -35,5 +35,5 @@
     <!-- RGB optical joint -->
     <joint name="${prefix}rgb_optical_joint" type="fixed">
-      <origin xyz="0.003 0 0" rpy="0 0 0" />
+      <origin xyz="0.003 0 0" rpy="${-M_PI/2} 0 ${-M_PI/2}" />
       <parent link="${prefix}link"/>
       <child link="${prefix}rgb_optical_link" />
@@ -41,13 +41,18 @@
 		<!-- ov5647 sensor for simulation -->
     <xacro:if value="${use_sim}">
-      <xacro:sensor_ov5647_gazebo/>
+      <xacro:sensor_ov5647_gazebo prefix="${prefix}" prefix_topic="${prefix_topic}"/>
     </xacro:if>
   </xacro:macro>
 <!-- - - - - - - - - - - - - - OV5647 GAZEBO - - - - - - - - - - - - - -->
-  <xacro:macro name="sensor_ov5647_gazebo">
+  <xacro:macro name="sensor_ov5647_gazebo" params="prefix prefix_topic">
     <gazebo reference="${prefix}link">
-      <sensor type="depth" name="${prefix}sensor">
+      <sensor name="${prefix}sensor" type="camera">
+        <pose>0 0 0 0 0 0</pose>
+        <update_rate>30</update_rate>
         <always_on>true</always_on>
-        <update_rate>30.0</update_rate>
+        <topic>${prefix_topic}/color/image_raw</topic>
+        <camera_info_topic>${prefix_topic}/color/camera_info</camera_info_topic>
+        <!-- Hack to set frame id for gazebo ros2 bridge. Ignore SDF warning -->
+        <gz_frame_id>${prefix}rgb_optical_link</gz_frame_id>
         <camera>
           <horizontal_fov>${60.0*M_PI/180.0}</horizontal_fov>
@@ -62,18 +67,4 @@
           </clip>
         </camera>
-        <plugin name="${prefix}controller" filename="libgazebo_ros_camera.so">
-          <cameraName>${prefix_topic}</cameraName>
-          <alwaysOn>true</alwaysOn>
-          <updateRate>0.0</updateRate>
-          <imageTopicName>rgb/image_raw</imageTopicName>
-          <cameraInfoTopicName>rgb/camera_info</cameraInfoTopicName>
-          <frameName>/${prefix}rgb_optical_link</frameName>
-          <hackBaseline>0.07</hackBaseline>
-          <distortion_k1>0.0</distortion_k1>
-          <distortion_k2>0.0</distortion_k2>
-          <distortion_k3>0.0</distortion_k3>
-          <distortion_t1>0.0</distortion_t1>
-          <distortion_t2>0.0</distortion_t2>
-        </plugin>
       </sensor>
     </gazebo>
