Commit message: base/description: Fix gazebo lidar scan

File: src/base/nano_atom_description/urdf/devices/ydlidar_x2.urdf.xacro (robot description, xacro)
@@ -2,5 +2,5 @@
 <robot name="sensor_ydlidar_x2" xmlns:xacro="http://www.ros.org/wiki/xacro">
 <!-- - - - - - - - - - - - - - RPLIDAR SENSOR - - - - - - - - - - - - - -->
-  <xacro:macro name ="sensor_ydlidar_x2" params="prefix prefix_topic:='front_laser/scan' use_sim gpu_sim='false' parent *origin">
+  <xacro:macro name ="sensor_ydlidar_x2" params="prefix prefix_topic:='front_laser/scan' use_sim gpu_sim='true' parent *origin">
     <link name="${prefix}link">
       <collision>
@@ -34,10 +34,11 @@
   </xacro:macro>
 <!-- - - - - - - - - - - - - - YDLIDAR GAZEBO - - - - - - - - - - - - - -->
-<xacro:macro name="sensor_ydlidar_x2_gazebo" params="prefix prefix_topic gpu_sim:=false">
+<xacro:macro name="sensor_ydlidar_x2_gazebo" params="prefix prefix_topic gpu_sim:=true">
   <xacro:if value="${gpu_sim}">
     <xacro:property name="ray_type" value="gpu_lidar"/>
   </xacro:if>
   <xacro:unless value="${gpu_sim}">
-    <xacro:property name="ray_type" value="gpu_lidar"/> <!-- lidar -->
+    <!-- CPU lidar not supported by gz sim yet. 'lidar'  -->
+    <xacro:property name="ray_type" value="gpu_lidar"/>
   </xacro:unless>
   <gazebo reference="${prefix}link">
@@ -52,6 +53,6 @@
         <scan>
           <horizontal>
-            <samples>360</samples>
-            <resolution>0.9</resolution>
+            <samples>400</samples>
+            <resolution>1</resolution>
             <min_angle>-3.14159</min_angle>
             <max_angle>3.14159</max_angle>
@@ -65,12 +66,12 @@
         </scan>
         <range>
-          <min>0.15</min>
-          <max>6.0</max>
-          <resolution>0.02</resolution>
+          <min>0.12</min>
+          <max>8.0</max>
+          <resolution>0.01</resolution>
         </range>
         <noise>
           <type>gaussian</type>
           <mean>0.0</mean>
-          <stddev>0.01</stddev>
+          <stddev>0.02</stddev>
         </noise>
       </lidar>
