Commit message: modules: Use substitutions for configurable params

File: modules/base/nano_atom_description/robots/nano_atom_std.urdf.xacro (robot description, xacro)
@@ -6,4 +6,5 @@
   <xacro:arg name="controller_sim_path" default="$(find ${nano_atom_control})/config/diff_controller.yaml" />
   <xacro:arg name="hardware_path"       default="$(find ${nano_atom_hardware})/config/hardware.yaml" />
+  <xacro:arg name="driver_uri"          default="/dev/ttyAMA_NANO_ATOM"/>
   <xacro:arg name="use_front_laser"     default="false" />
   <xacro:arg name="use_front_camera"    default="false" />
@@ -36,5 +37,6 @@
       use_sim="$(arg use_sim)"
       controller_sim_path="$(arg controller_sim_path)"
-      hardware_path="$(arg hardware_path)"/>
+      hardware_path="$(arg hardware_path)"
+      driver_uri="$(arg driver_uri)"/>
 <!-- - - - - - - - - - - - - - - BASE DEFINITION  - - - - - - - - - - - - - -->
   <!-- base_footprint definition -->
@@ -55,8 +57,9 @@
 	<xacro:property name="wheel_offset_y" value="0.04519" />
 	<xacro:property name="wheel_offset_z" value="0.005" />
-  <xacro:rubber_wheel prefix="$(arg prefix)right_" parent ="$(arg base_frame)" type="right">
+  <!-- Joint names are local to the URDF/ros2_control instance and do not require /robot namespace -->
+  <xacro:rubber_wheel prefix="right_" parent ="$(arg base_frame)" type="right">
   	<origin xyz="${wheel_offset_x} -${wheel_offset_y} +${wheel_offset_z}" rpy="0 0 0"/>
   </xacro:rubber_wheel>
-  <xacro:rubber_wheel prefix="$(arg prefix)left_" parent ="$(arg base_frame)" type="left">
+  <xacro:rubber_wheel prefix="left_" parent ="$(arg base_frame)" type="left">
   	<origin xyz="${wheel_offset_x} +${wheel_offset_y} +${wheel_offset_z}" rpy="0 0 0"/>
   </xacro:rubber_wheel>

File: modules/base/nano_atom_description/urdf/controllers/diff.ros2_control.urdf.xacro (robot description, xacro)
@@ -2,5 +2,5 @@
 <robot xmlns:xacro="http://wiki.ros.org/xacro">
   <!--Plugin used to connect ROS2 with hardware or simulation -->
-  <xacro:macro name="diff_ros2_control" params="robot_id prefix use_sim controller_sim_path hardware_path">
+  <xacro:macro name="diff_ros2_control" params="robot_id prefix use_sim controller_sim_path hardware_path driver_uri">
     <xacro:macro name="ros2_joint" params="interface jmin jmax name">
       <joint name="${name}">
@@ -23,11 +23,12 @@
           <param name="left_wheel_joint_name">${hw_param['left_wheel_joint']}</param>
           <param name="right_wheel_joint_name">${hw_param['right_wheel_joint']}</param>
-          <param name="serial_port">${hw_param['serial_port']}</param>
+          <param name="serial_port">${driver_uri}</param>
           <param name="serial_baudrate">${hw_param['serial_baudrate']}</param>
           <param name="serial_timeout">${hw_param['serial_timeout']}</param>
           <param name="resolution">${hw_param['resolution']}</param>
         </hardware>
-        <xacro:ros2_joint interface="velocity" jmin="-5" jmax="5" name="${prefix}left_wheel_joint"/>
-        <xacro:ros2_joint interface="velocity" jmin="-5" jmax="5" name="${prefix}right_wheel_joint"/>
+        <!-- Joint names are local to the URDF/ros2_control instance and do not require /robot namespace -->
+        <xacro:ros2_joint interface="velocity" jmin="-5" jmax="5" name="left_wheel_joint"/>
+        <xacro:ros2_joint interface="velocity" jmin="-5" jmax="5" name="right_wheel_joint"/>
       </ros2_control>
     </xacro:unless>
@@ -50,6 +51,7 @@
           <plugin>gz_ros2_control/GazeboSimSystem</plugin>
         </hardware>
-        <xacro:ros2_joint interface="velocity" jmin="-5" jmax="5" name="${prefix}left_wheel_joint"/>
-        <xacro:ros2_joint interface="velocity" jmin="-5" jmax="5" name="${prefix}right_wheel_joint"/>
+        <!-- Joint names are local to the URDF/ros2_control instance and do not require /robot namespace -->
+        <xacro:ros2_joint interface="velocity" jmin="-5" jmax="5" name="left_wheel_joint"/>
+        <xacro:ros2_joint interface="velocity" jmin="-5" jmax="5" name="right_wheel_joint"/>
       </ros2_control>
     </xacro:if>

Commit message: base/description: Fix wheel namespaces

File: modules/base/nano_atom_description/robots/nano_atom_std.urdf.xacro (robot description, xacro)
@@ -57,9 +57,8 @@
 	<xacro:property name="wheel_offset_y" value="0.04519" />
 	<xacro:property name="wheel_offset_z" value="0.005" />
-  <!-- Joint names are local to the URDF/ros2_control instance and do not require /robot namespace -->
-  <xacro:rubber_wheel prefix="right_" parent ="$(arg base_frame)" type="right">
+  <xacro:rubber_wheel link_prefix="$(arg prefix)right_" joint_prefix="right_" parent ="$(arg base_frame)" type="right">
   	<origin xyz="${wheel_offset_x} -${wheel_offset_y} +${wheel_offset_z}" rpy="0 0 0"/>
   </xacro:rubber_wheel>
-  <xacro:rubber_wheel prefix="left_" parent ="$(arg base_frame)" type="left">
+  <xacro:rubber_wheel link_prefix="$(arg prefix)left_" joint_prefix="left_" parent ="$(arg base_frame)" type="left">
   	<origin xyz="${wheel_offset_x} +${wheel_offset_y} +${wheel_offset_z}" rpy="0 0 0"/>
   </xacro:rubber_wheel>

File: modules/base/nano_atom_description/urdf/wheels/rubber_wheel.urdf.xacro (robot description, xacro)
@@ -34,14 +34,15 @@
   </xacro:macro>
 <!-- - - - - - - - - - - - - - WHEEL DEFINITION - - - - - - - - - - - - - -->
-  <xacro:macro name ="rubber_wheel" params = "prefix parent *origin type">
+  <xacro:macro name ="rubber_wheel" params = "link_prefix joint_prefix parent *origin type">
     <!-- wheel & base joint-->
-    <joint name="${prefix}wheel_joint" type="continuous">
+    <!-- Joint names are local to the URDF/ros2_control instance and do not require /robot namespace -->
+    <joint name="${joint_prefix}wheel_joint" type="continuous">
       <xacro:insert_block name ="origin" />
       <parent link="${parent}" />
-      <child link="${prefix}wheel_link" />
+      <child link="${link_prefix}wheel_link" />
       <axis xyz="0 1 0" />
     </joint>
     <!-- wheel link -->
-    <link name="${prefix}wheel_link">
+    <link name="${link_prefix}wheel_link">
       <inertial>
         <xacro:origin_selector wheel = "${type}" />
